File: HybridRocket2017_nose.kicad_pcb (KiCad board)
At the start: 2 copper layers, 50 x 46 mm, 37 parts, among them CON1 SD_Card, P1 Switch, P2 PowerIN, P3 DEBUG, P4 STLINK, U1 LT1963A-3.3, U2 STM32F4xxRx, U3 MP3V5050, Y1 XTAL

Commit message: 製作中にコミットするの忘れてた
Parts:
- removed ? (x2): MountingHole_3.2mm_M3, Mounting_Holes:MountingHole_3.2mm_M3
- added REF**: MountingHole_2.2mm_M2, Mounting_Holes:MountingHole_2.2mm_M2, F.Cu at (95.0, 92.0)
- added REF**: MountingHole_2.2mm_M2, Mounting_Holes:MountingHole_2.2mm_M2, F.Cu at (55.0, 92.0)
Routing:
- net GND: track 505.4 -> 481.3 mm, vias 71 -> 72
- net (no net): track 0.00 -> 7.52 mm, vias 0 -> 1
- net Net-(C2-Pad2): track 46.8 -> 45.7 mm
Other:
- board size 50 x 46 mm -> 50 x 40 mm
