File: HybridRocket2017_nose.sch (KiCad schematic (older format))
At the start: 35 parts, among them CON1 SD_Card, P1 Switch, P2 PowerIN, P3 DEBUG, P4 STLINK, U1 LT1963A-3.3, U2 STM32F4xxRx, U3 MP3V5050, Y1 XTAL

Commit message: 製作中にコミットするの忘れてた
Parts:
- C2: value 10u -> 1u
Changed lines of the file:
@@
 P 2350 2450
 F 0 "C2" H 2360 2520 50  0000 L CNN
-F 1 "10u" H 2360 2370 50  0000 L CNN
+F 1 "1u" H 2360 2370 50  0000 L CNN
 F 2 "Capacitors_SMD:C_0805" H 2350 2450 50  0001 C CNN
 F 3 "" H 2350 2450 50  0000 C CNN
